File: E1041 - PCB, Driver Board/ethernet.kicad_sch (KiCad schematic)
At the start: 45 parts, among them J3 74984104400, U1 TPS2372, U11 VCB48_SO-3WR3, U4 LAN8720A

Commit message: Added 'Part Number' in schematic, no design change
Parts:
- C2: value 100uF -> 10uF; Part Number (none) -> 865060845002; Voltage (none) -> 100V
- C4, C5: Voltage (none) -> 100V
- D1, D2: Part Number (none) -> CDBHM220L
- D3: Part Number (none) -> SMAJ58A
- J3: Part Number (none) -> 74984104400
- L3, L4: Part Number (none) -> BLM21AG102SN1D
- U1: Part Number (none) -> TPS2372
- U11: Part Number (none) -> VCB4812SO-3WR3
- U4: Part Number (none) -> LAN8720Ar
